Commit message: Warehouse model working, sensor plugins working, there is very significant lag between cmd_vels being sent and the robot moving in sim

File: simulation_ws/install/simulation_app/share/simulation_app/urdf/2WD_Rover.gazebo.xacro (robot description, xacro)
@@ -1,85 +1,36 @@
 <?xml version="1.0"?>
 <robot name="rover_sim" xmlns:xacro="http://ros.org/wiki/xacro">
-  <xacro:arg name="laser_visual"  default="false"/>
-  <xacro:arg name="camera_visual" default="false"/>
-  <xacro:arg name="imu_visual"    default="false"/>
   <gazebo reference="base_link">
-    <material>Gazebo/DarkGrey</material>
+    <material>Gazebo/FlatBlack</material>
+  </gazebo>
+  <gazebo reference="sheetmetal_link">
+    <material>Gazebo/FlatBlack</material>
   </gazebo>
   <gazebo reference="wheel_left_link">
-    <mu1>0.1</mu1>
-    <mu2>0.1</mu2>
-    <kp>500000.0</kp>
-    <kd>10.0</kd>
-    <minDepth>0.001</minDepth>
-    <maxVel>0.1</maxVel>
-    <fdir1>1 0 0</fdir1>
-    <material>Gazebo/White</material>
+    <mu1>0.7</mu1>
+    <mu2>1.0</mu2>
+    <kp>300000.0</kp>
+    <material>Gazebo/Black</material>
   </gazebo>
   <gazebo reference="wheel_right_link">
+    <mu1>0.7</mu1>
+    <mu2>1.0</mu2>
+    <kp>300000.0</kp>
+    <material>Gazebo/Black</material>
+  </gazebo>
+  <gazebo reference="caster_back_left_link">
     <mu1>0.1</mu1>
-    <mu2>0.1</mu2>
-    <kp>500000.0</kp>
-    <kd>10.0</kd>
-    <minDepth>0.001</minDepth>
-    <maxVel>0.1</maxVel>
-    <fdir1>1 0 0</fdir1>
-    <material>Gazebo/White</material>
-  </gazebo>
-  <gazebo reference="sheetmetal_link">
-    <mu1>0.1</mu1>
-    <mu2>0.1</mu2>
-    <kp>1000000.0</kp>
-    <kd>100.0</kd>
-    <minDepth>0.001</minDepth>
-    <maxVel>1.0</maxVel>
-    <material>Gazebo/White</material>
+    <mu2>0.6</mu2>
+    <kp>200000.0</kp>
+    <material>Gazebo/Grey</material>
   </gazebo>
   <gazebo reference="caster_back_right_link">
     <mu1>0.1</mu1>
-    <mu2>0.1</mu2>
-    <kp>1000000.0</kp>
-    <kd>100.0</kd>
-    <minDepth>0.001</minDepth>
-    <maxVel>1.0</maxVel>
-    <material>Gazebo/FlatBlack</material>
-  </gazebo>
-  <gazebo reference="caster_back_left_link">
-    <mu1>0.1</mu1>
-    <mu2>0.1</mu2>
-    <kp>1000000.0</kp>
-    <kd>100.0</kd>
-    <minDepth>0.001</minDepth>
-    <maxVel>1.0</maxVel>
-    <material>Gazebo/FlatBlack</material>
-  </gazebo>
-  <gazebo reference="imu_link">
-    <sensor type="imu" name="imu">
-      <always_on>true</always_on>
-      <visualize>$(arg imu_visual)</visualize>
-    </sensor>
+    <mu2>0.6</mu2>
+    <kp>200000.0</kp>
     <material>Gazebo/Grey</material>
   </gazebo>
-  <gazebo>
-    <plugin name="turtlebot3_waffle_controller" filename="libgazebo_ros_diff_drive.so">
-      <commandTopic>cmd_vel</commandTopic>
-      <odometryTopic>odom</odometryTopic>
-      <odometryFrame>odom</odometryFrame>
-      <odometrySource>world</odometrySource>
-      <publishOdomTF>true</publishOdomTF>
-      <robotBaseFrame>base_footprint</robotBaseFrame>
-      <publishWheelTF>false</publishWheelTF>
-      <publishTf>true</publishTf>
-      <publishWheelJointState>true</publishWheelJointState>
-      <legacyMode>false</legacyMode>
-      <updateRate>30</updateRate>
-      <leftJoint>wheel_left_joint</leftJoint>
-      <rightJoint>wheel_right_joint</rightJoint>
-      <wheelSeparation>0.287</wheelSeparation>
-      <wheelDiameter>0.066</wheelDiameter>
-      <wheelAcceleration>1</wheelAcceleration>
-      <wheelTorque>10</wheelTorque>
-      <rosDebugLevel>na</rosDebugLevel>
-    </plugin>
+  <gazebo reference="plate_link">
+    <material>Gazebo/GreyTransparent</material>
   </gazebo>
   <gazebo>
@@ -111,9 +62,11 @@
     </plugin>
   </gazebo>
-  <gazebo reference="base_scan">
+  <gazebo reference="cpu_link">
+    <material>Gazebo/DarkGrey</material>
+  </gazebo>
+  <gazebo reference="lidar_link">
     <material>Gazebo/FlatBlack</material>
     <sensor type="ray" name="lds_lfcd_sensor">
       <pose>0 0 0 0 0 0</pose>
-      <visualize>$(arg laser_visual)</visualize>
       <update_rate>5</update_rate>
       <ray>
@@ -139,50 +92,38 @@
       <plugin name="gazebo_ros_lds_lfcd_controller" filename="libgazebo_ros_laser.so">
         <topicName>scan</topicName>
-        <frameName>base_scan</frameName>
+        <frameName>lidar_link</frameName>
       </plugin>
     </sensor>
   </gazebo>
-  <gazebo reference="camera_rgb_frame">
-    <sensor type="depth" name="realsense_R200">
-      <always_on>true</always_on>
-      <visualize>$(arg camera_visual)</visualize>
-      <camera>
-          <horizontal_fov>1.3439</horizontal_fov>
-          <image>
-              <width>1920</width>
-              <height>1080</height>
-              <format>R8G8B8</format>
-          </image>
-          <depth_camera></depth_camera>
-          <clip>
-              <near>0.03</near>
-              <far>100</far>
-          </clip>
-      </camera>
-      <plugin name="camera_controller" filename="libgazebo_ros_openni_kinect.so">
-        <baseline>0.2</baseline>
-        <alwaysOn>true</alwaysOn>
-        <updateRate>30.0</updateRate>
-        <cameraName>camera</cameraName>
-        <frameName>camera_rgb_optical_frame</frameName>
-        <imageTopicName>rgb/image_raw</imageTopicName>
-        <depthImageTopicName>depth/image_raw</depthImageTopicName>
-        <pointCloudTopicName>depth/points</pointCloudTopicName>
-        <cameraInfoTopicName>rgb/camera_info</cameraInfoTopicName>
-        <depthImageCameraInfoTopicName>depth/camera_info</depthImageCameraInfoTopicName>
-        <pointCloudCutoff>0.4</pointCloudCutoff>
-            <hackBaseline>0.07</hackBaseline>
-            <distortionK1>0.0</distortionK1>
-            <distortionK2>0.0</distortionK2>
-            <distortionK3>0.0</distortionK3>
-            <distortionT1>0.0</distortionT1>
-            <distortionT2>0.0</distortionT2>
-        <CxPrime>0.0</CxPrime>
-        <Cx>0.0</Cx>
-        <Cy>0.0</Cy>
-        <focalLength>0</focalLength>
-        <hackBaseline>0</hackBaseline>
-      </plugin>
-    </sensor>
+  <gazebo>
+    <plugin name="turtlebot3_waffle_controller" filename="libgazebo_ros_diff_drive.so">
+      <commandTopic>cmd_vel</commandTopic>
+      <odometryTopic>odom</odometryTopic>
+      <odometryFrame>odom</odometryFrame>
+      <odometrySource>world</odometrySource>
+      <publishOdomTF>true</publishOdomTF>
+      <robotBaseFrame>base_footprint</robotBaseFrame>
+      <publishWheelTF>false</publishWheelTF>
+      <publishTf>true</publishTf>
+      <publishWheelJointState>true</publishWheelJointState>
+      <legacyMode>false</legacyMode>
+      <updateRate>30</updateRate>
+      <leftJoint>wheel_left_joint</leftJoint>
+      <rightJoint>wheel_right_joint</rightJoint>
+      <wheelSeparation>0.287</wheelSeparation>
+      <wheelDiameter>0.066</wheelDiameter>
+      <wheelAcceleration>1</wheelAcceleration>
+      <wheelTorque>10</wheelTorque>
+      <rosDebugLevel>na</rosDebugLevel>
+    </plugin>
+  </gazebo>
+  <gazebo>
+    <plugin name="gazebo_joint_publisher" filename="libgazebo_ros_joint_state_publisher.so">
+      <joint_name>wheel_left_joint</joint_name>
+      <joint_name>wheel_right_joint</joint_name>
+      <joint_name>caster_back_left_joint</joint_name>
+      <joint_name>caster_back_right_joint</joint_name>
+      <update_rate>30.0</update_rate>
+    </plugin>
   </gazebo>
 </robot>

File: simulation_ws/install/simulation_app/share/simulation_app/urdf/rover.urdf.xacro (robot description, xacro)
@@ -1,11 +1,11 @@
 <?xml version="1.0" ?>
 <robot name="2WD_rover_robotics" xmlns:xacro="http://ros.org/wiki/xacro">
+  <xacro:include filename="$(find simulation_app)/urdf/common_properties.xacro"/>
   <xacro:include filename="$(find simulation_app)/urdf/2WD_Rover.gazebo.xacro"/>
-  <xacro:include filename="$(find simulation_app)/urdf/common_properties.xacro"/>
   <link name="base_footprint"/>
   <joint name="base_joint" type="fixed">
     <parent link="base_footprint"/>
-    <child link="base_link" />
-    <origin xyz="0 0 0.01" rpy="0 0 0"/>
+    <child link="base_link"/>
+    <origin xyz="0 0 0.12" rpy="0 0 0"/>
   </joint>
   <link name="base_link">
@@ -14,19 +14,24 @@
       <geometry>
         <mesh filename="package://simulation_app/meshes/2WD_OpenRover.stl" scale="1 1 1"/>
-      </geometry>
-      <material name="light_black"/>
-    </visual>
-    <collision>
-      <origin xyz="-0.14 0 0" rpy="0 0 0"/>
+      <!--
+      <origin xyz="-0.142 0 0" rpy="0 0 0"/>
       <geometry>
         <box size="0.42 0.25 0.12"/>
-      </geometry>
-    </collision>
-    <inertial>
-      <origin xyz="0 0 0" rpy="0 0 0"/>
-      <mass value="1.3729096e+00"/>
-      <inertia ixx="8.7002718e-03" ixy="-4.7576583e-05" ixz="1.1160499e-04"
-               iyy="8.6195418e-03" iyz="-3.5422299e-06"
-               izz="1.4612727e-02" />
+        -->
+      </geometry>
+      <material name="dark"/>
+    </visual>
+    <collision>
+      <origin xyz="-0.142 0 0" rpy="0 0 0"/>
+      <geometry>
+        <box size="0.42 0.25 0.12"/>
+      </geometry>
+    </collision>
+    <inertial>
+      <origin xyz="-0.142 0 0" rpy="0 0 0" />
+      <mass value="7.5" />
+      <inertia ixx="4.806e-2"
+               ixy="0.0" iyy="1.193e-1"
+               ixz="0.0" iyz="0.0" izz="1.493e-1" />
     </inertial>
   </link>
@@ -42,20 +47,25 @@
       <geometry>
         <mesh filename="package://simulation_app/meshes/left_wheel.stl" scale="1 1 1"/>
-      </geometry>
-      <material name="light_black"/>
-    </visual>
-    <collision>
-      <origin xyz="0 0 0" rpy="0 0 0"/>
-      <geometry>
-        <cylinder length="0.07" radius="0.12"/>
-      </geometry>
-    </collision>
-    <inertial>
-      <origin xyz="0 0 0" />
-      <mass value="2.8498940e-02" />
-      <inertia ixx="1.1175580e-05" ixy="-4.2369783e-11" ixz="-5.9381719e-09"
-               iyy="1.1192413e-05" iyz="-1.4400107e-11"
-               izz="2.0712558e-05" />
-      </inertial>
+      <!--
+      <origin xyz="0 0 0" rpy="0 0 3.14"/>
+      <geometry>
+        <cylinder length="0.07" radius="0.12"/>
+        -->
+      </geometry>
+      <material name="black"/>
+    </visual>
+    <collision>
+      <origin xyz="0 0 0" rpy="0 0 3.14"/>
+      <geometry>
+        <cylinder length="0.07" radius="0.12"/>
+      </geometry>
+    </collision>
+    <inertial>
+      <origin xyz="0 0 0" rpy="0 0 3.14" />
+      <mass value="1.525" />
+      <inertia ixx="6.723e-3"
+               ixy="0.0" iyy="6.723e-3"
+               ixz="0.0" iyz="0.0" izz="1.220e-2" />
+    </inertial>
   </link>
   <joint name="wheel_right_joint" type="continuous">
@@ -70,19 +80,24 @@
       <geometry>
         <mesh filename="package://simulation_app/meshes/right_wheel.stl" scale="1 1 1"/>
-      </geometry>
-      <material name="light_black"/>
-    </visual>
-    <collision>
-      <origin xyz="0 0 0" rpy="0 0 0"/>
-      <geometry>
-        <cylinder length="0.07" radius="0.12"/>
-      </geometry>
-    </collision>
-    <inertial>
-      <origin xyz="0 0 0" />
-      <mass value="2.8498940e-02" />
-      <inertia ixx="1.1175580e-05" ixy="-4.2369783e-11" ixz="-5.9381719e-09"
-               iyy="1.1192413e-05" iyz="-1.4400107e-11"
-               izz="2.0712558e-05" />
+      <!--
+      <origin xyz="0 0 0" rpy="0 0 0"/>
+      <geometry>
+        <cylinder length="0.07" radius="0.12"/>
+        -->
+      </geometry>
+      <material name="black"/>
+    </visual>
+    <collision>
+      <origin xyz="0 0 0" rpy="0 0 0"/>
+      <geometry>
+        <cylinder length="0.07" radius="0.12"/>
+      </geometry>
+    </collision>
+    <inertial>
+      <origin xyz="0 0 0" rpy="0 0 0" />
+      <mass value="1.525" />
+      <inertia ixx="6.723e-3"
+               ixy="0.0" iyy="6.723e-3"
+               ixz="0.0" iyz="0.0" izz="1.220e-2" />
     </inertial>
   </link>
@@ -97,33 +112,150 @@
       <geometry>
         <mesh filename="package://simulation_app/meshes/sheetmetal_part.stl" scale="1 1 1"/>
+      <!--
+      <origin xyz="0 0 0" rpy="0 0 0"/>
+      <geometry>
+        <box size="0.065 0.4 0.008"/>
+        -->
+      </geometry>
+      <material name="dark"/>
+    </visual>
+    <collision>
+      <origin xyz="-0.007 0 0" rpy="0 0 0"/>
+      <geometry>
+        <box size="0.065 0.4 0.008"/>
+      </geometry>
+    </collision>
+    <inertial>
+      <origin xyz="0 0 0" />
+      <mass value="0.6" />
+      <inertia ixx="8.020e-3"
+               ixy="0.0" iyy="2.313e-4"
+               ixz="0.0" iyz="0.0" izz="8.211e-3" />
+    </inertial>
+  </link>
+  <joint name="plate_link_joint" type="fixed">
+    <parent link="base_link"/>
+    <child link="plate_link"/>
+    <origin xyz="-0.1365 0 0.127" rpy="0 0 0"/>
+  </joint>
+  <link name="plate_link">
+    <visual>
+      <origin xyz="0 0 0" rpy="0 0 0"/>
+      <geometry>
+        <box size="0.381 0.254 0.005"/>
+      </geometry>
+      <material name="acrylic"/>
+    </visual>
+    <inertial>
+      <origin xyz="0 0 0" />
+      <mass value="0.65" />
+      <inertia ixx="3.496e-3"
+               ixy="0.0" iyy="7.864e-3"
+               ixz="0.0" iyz="0.0" izz="1.136e-2" />
+    </inertial>
+  </link>
+  <joint name="imu_link_joint" type="fixed">
+    <parent link="plate_link"/>
+    <child link="imu_link"/>
+    <origin xyz="0.1365 0 0.0026" rpy="0 0 0"/>
+  </joint>
+  <link name="imu_link">
+    <visual>
+      <origin xyz="0 0 0" rpy="0 0 0"/>
+      <geometry>
+        <box size="0.01 0.01 0.002"/>
+      </geometry>
+      <material name="blue"/>
+    </visual>
+    <inertial>
+      <origin xyz="0 0 0" />
+      <mass value="0.04" />
+      <inertia ixx="3.467e-7"
+               ixy="0.0" iyy="3.467e-7"
+               ixz="0.0" iyz="0.0" izz="6.667e-7" />
+    </inertial>
+  </link>
+  <joint name="cpu_link_joint" type="fixed">
+    <parent link="plate_link"/>
+    <child link="cpu_link"/>
+    <origin xyz="-0.0032 0 0.0275" rpy="0 0 0"/>
+  </joint>
+  <link name="cpu_link">
+    <visual>
+      <origin xyz="0 0 0" rpy="0 0 0"/>
+      <geometry>
+        <box size="0.111 0.117 0.05"/>
       </geometry>
       <material name="light_black"/>
     </visual>
-    <collision>
-      <origin xyz="-0.05 0 0" rpy="0 0 0"/>
-      <geometry>
-        <box size="0.065 0.3 0.008"/>
-      </geometry>
-    </collision>
-  </link>
-  <joint name="imu_link_joint" type="fixed">
-    <parent link="base_link"/>
-    <child link="imu_link"/>
-    <origin xyz="0 0 0" rpy="0 0 0"/>
-  </joint>
-  <link name="imu_link">
-    <visual>
-      <origin xyz="0 0 0" rpy="0 0 0"/>
-      <geometry>
-        <box size="0.01 0.01 0.002"/>
+    <inertial>
+      <origin xyz="0 0 0" />
+      <mass value="0.64" />
+      <inertia ixx="8.634e-4"
+               ixy="0.0" iyy="7.905e-4"
+               ixz="0.0" iyz="0.0" izz="1.387e-3" />
+    </inertial>
+  </link>
+  <joint name="lidar_link_joint" type="fixed">
+    <parent link="cpu_link"/>
+    <child link="lidar_link"/>
+    <origin xyz="0 0 0.0488" rpy="0 0 0"/>
+  </joint>
+  <link name="lidar_link">
+    <visual>
+      <origin xyz="0 0 0" rpy="0 0 0"/>
+      <geometry>
+        <cylinder length="0.0476" radius="0.0381"/>
       </geometry>
       <material name="light_black"/>
     </visual>
+    <inertial>
+      <origin xyz="0 0 0" />
+      <mass value="0.220" />
+      <inertia ixx="1.214e-4"
+               ixy="0.0" iyy="1.214e-4"
+               ixz="0.0" iyz="0.0" izz="1.597e-4" />
+    </inertial>
+  </link>
+  <joint name="caster_back_left_joint" type="continuous">
+    <parent link="sheetmetal_link"/>
+    <child link="caster_back_left_link"/>
+    <origin xyz="-0.01 0.17 -0.01" rpy="0 0 0"/>
+    <axis xyz="0 0 1"/>
+    <dynamics damping="0.1" friction="0.01"/>
+  </joint>
+  <link name="caster_back_left_link">
+    <visual>
+      <origin xyz="0 0 0" rpy="1.57 0 3.14"/>
+      <geometry>
+        <mesh filename="package://simulation_app/meshes/left_caster_wheel.stl" scale="1 1 1"/>
+      <!--
+      <origin xyz="-0.028 0 -0.065" rpy="1.57 0 3.14"/>
+      <geometry>
+        <cylinder length="0.035" radius="0.048"/>
+        -->
+      </geometry>
+      <material name="grey"/>
+    </visual>
+    <collision>
+      <origin xyz="-0.035 0 -0.065" rpy="1.57 0 3.14"/>
+      <geometry>
+        <cylinder length="0.0035" radius="0.05"/>
+      </geometry>
+    </collision>
+    <inertial>
+      <origin xyz="-0.005 0 -0.03" />
+      <mass value="0.41" />
+      <inertia ixx="3.841e-4"
+               ixy="0.0" iyy="4.592e-4"
+               ixz="0.0" iyz="0.0" izz="2.135e-4" />
+    </inertial>
   </link>
   <joint name="caster_back_right_joint" type="continuous">
-    <parent link="base_link"/>
+    <parent link="sheetmetal_link"/>
     <child link="caster_back_right_link"/>
-    <origin xyz="-0.36 -0.17 -0.01" rpy="0 0 0"/>
-    <axis xyz="0 0 1"/>
+    <origin xyz="-0.01 -0.17 -0.01" rpy="0 0 0"/>
+    <axis xyz="0 0 1"/>
+    <dynamics damping="0.1" friction="0.01"/>
   </joint>
   <link name="caster_back_right_link">
@@ -132,47 +264,24 @@
       <geometry>
         <mesh filename="package://simulation_app/meshes/right_caster_wheel.stl" scale="1 1 1"/>
-      </geometry>
-      <material name="light_black"/>
-    </visual>
-    <collision>
-      <origin xyz="-0.028 0 -0.065" rpy="1.57 0 0"/>
+      <!--
+      <origin xyz="-0.028 0 -0.065" rpy="1.57 0 3.14"/>
       <geometry>
         <cylinder length="0.035" radius="0.048"/>
-      </geometry>
-    </collision>
-    <inertial>
-      <origin xyz="0 0 0" />
-      <mass value="0.005" />
-      <inertia ixx="0.001" ixy="0.0" ixz="0.0"
-               iyy="0.001" iyz="0.0"
-               izz="0.001" />
-    </inertial>
-  </link>
-  <joint name="caster_back_left_joint" type="continuous">
-    <parent link="base_link"/>
-    <child link="caster_back_left_link"/>
-    <origin xyz="-0.36 0.17 -0.01" rpy="0 0 0"/>
-    <axis xyz="0 0 1"/>
-  </joint>
-  <link name="caster_back_left_link">
-    <visual>
-      <origin xyz="0 0 0" rpy="1.57 0 3.14"/>
-      <geometry>
-        <mesh filename="package://simulation_app/meshes/left_caster_wheel.stl" scale="1 1 1"/>
-      </geometry>
-      <material name="light_black"/>
-    </visual>
-    <collision>
-      <origin xyz="-0.028 0 -0.065" rpy="1.57 0 0"/>
-      <geometry>
-        <cylinder length="0.035" radius="0.048"/>
-      </geometry>
-    </collision>
-    <inertial>
-      <origin xyz="0 0 0" />
-      <mass value="0.005" />
-      <inertia ixx="0.001" ixy="0.0" ixz="0.0"
-               iyy="0.001" iyz="0.0"
-               izz="0.001" />
+        -->
+      </geometry>
+      <material name="grey"/>
+    </visual>
+    <collision>
+      <origin xyz="-0.035 0 -0.065" rpy="1.57 0 3.14"/>
+      <geometry>
+        <cylinder length="0.0035" radius="0.05"/>
+      </geometry>
+    </collision>
+    <inertial>
+      <origin xyz="-0.005 0 -0.03" />
+      <mass value="0.41" />
+      <inertia ixx="3.841e-4"
+               ixy="0.0" iyy="4.592e-4"
+               ixz="0.0" iyz="0.0" izz="2.135e-4" />
     </inertial>
   </link>
