Commit message: added imu sensor with gravity

File: simulation_ws/src/simulation_app/urdf/rover.urdf.xacro (robot description, xacro)
@@ -158,5 +158,5 @@
     <parent link="plate_link"/>
     <child link="imu_link"/>
-    <origin xyz="0.1365 0 0.0026" rpy="0 0 0"/>
+    <origin xyz="0.1365 0 0.0026" rpy="3.14 0 0"/>
   </joint>
   <link name="imu_link">
